Commit message: conditional mock component

File: my_robot_description/urdf/mobile_base.ros2_control.xacro (robot description, xacro)
@@ -3,10 +3,15 @@
   <ros2_control name="MobileBase" type="system">
     <hardware>
-      <!-- <plugin>mock_components/GenericSystem</plugin>
-      <param name="calculate_dynamics">true</param> -->
-      <plugin>mobile_base_hardware/MobileBaseHardwareInterface</plugin>
-      <param name="left_motor_id">10</param>
-      <param name="right_motor_id">20</param>
-      <param name="dynamixel_port">/dev/ttyACM0</param>
+      <xacro:property name="mock_mobile_base_hardware" value="true" />
+      <xacro:if value="${mock_mobile_base_hardware}">
+        <plugin>mock_components/GenericSystem</plugin>
+        <param name="calculate_dynamics">true</param>
+      </xacro:if>
+      <xacro:unless value="${mock_mobile_base_hardware}">
+        <plugin>mobile_base_hardware/MobileBaseHardwareInterface</plugin>
+        <param name="left_motor_id">10</param>
+        <param name="right_motor_id">20</param>
+        <param name="dynamixel_port">/dev/ttyACM0</param>
+      </xacro:unless>
     </hardware>
     <joint name="base_right_wheel_joint">

Commit message: additional hardware and controller lesson

File: my_robot_description/urdf/mobile_base.ros2_control.xacro (robot description, xacro)
@@ -3,4 +3,5 @@
   <ros2_control name="MobileBase" type="system">
     <hardware>
+      <!-- change this property to mock or not the mobile base hardware -->
       <xacro:property name="mock_mobile_base_hardware" value="true" />
       <xacro:if value="${mock_mobile_base_hardware}">

File: my_robot_description/urdf/my_robot.urdf.xacro (robot description, xacro)
@@ -5,12 +5,13 @@
   <xacro:include filename="mobile_base.xacro" />
   <xacro:include filename="mobile_base.ros2_control.xacro" />
+  <xacro:include filename="arm.xacro" />
+  <xacro:include filename="arm.ros2_control.xacro" />
   <!-- <xacro:include filename="mobile_base_gazebo.xacro" /> -->
-  <!-- <xacro:include filename="arm.xacro" /> -->
   <!-- <xacro:include filename="arm_gazebo.xacro" /> -->
   <!-- <xacro:include filename="camera.xacro" /> -->
-  <!-- <joint name="mobile_base_arm_joint" type="fixed">
+  <joint name="mobile_base_arm_joint" type="fixed">
     <parent link="base_link" />
     <child link="arm_base_link" />
     <origin xyz="${base_length / 4} 0 ${base_height}" rpy="0 0 0" />
-  </joint> -->
+  </joint>
 </robot>
